File: fotm-sign.kicad_sch (KiCad schematic)
At the start: 1 part, among them J1 Conn_01x03

Commit message: tweaks
Parts:
- J1: now not fitted
Changed lines of the file:
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@@
 		(on_board yes)
 		(in_pos_files yes)
-		(dnp no)
+		(dnp yes)
 		(fields_autoplaced yes)
 		(property "Reference" "J1"
