File: letter.kicad_sch (KiCad schematic)
At the start: 20 parts, among them U1 SK6805SIDE-G-003, U10 SK6805SIDE-G-003, U2 SK6805SIDE-G-003, U3 SK6805SIDE-G-003, U4 SK6805SIDE-G-003, U5 SK6805SIDE-G-003, U6 SK6805SIDE-G-003, U7 SK6805SIDE-G-003, U8 SK6805SIDE-G-003, U9 SK6805SIDE-G-003

Commit message: tweaks
Parts:
- C1, C10, C2, C3, C4, C5, C6, C7, C8, C9: LCSC Part (none) -> A
Changed lines of the file:
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@@
 			)
 		)
+		(property "LCSC Part" "A"
+			(at 80.01 68.58 90)
+			(hide yes)
+			(show_name no)
+			(do_not_autoplace no)
+			(effects
+				(font
+					(size 1.27 1.27)
+				)
+			)
+		)
 		(pin "2"
 		)
@@
 			)
 		)
+		(property "LCSC Part" "A"
+			(at 109.22 29.21 0)
+			(hide yes)
+			(show_name no)
+			(do_not_autoplace no)
+			(effects
+				(font
+					(size 1.27 1.27)
+				)
+			)
+		)
 		(pin "2"
 		)
@@
 			)
 		)
+		(property "LCSC Part" "A"
+			(at 148.59 58.42 90)
+			(hide yes)
+			(show_name no)
+			(do_not_autoplace no)
+			(effects
+				(font
+					(size 1.27 1.27)
+				)
+			)
+		)
 		(pin "2"
 		)
@@
 			)
 		)
+		(property "LCSC Part" "A"
+			(at 119.38 110.49 0)
+			(hide yes)
+			(show_name no)
+			(do_not_autoplace no)
+			(effects
+				(font
+					(size 1.27 1.27)
+				)
+			)
+		)
 		(pin "2"
 		)
@@
 			)
 		)
+		(property "LCSC Part" "A"
+			(at 121.92 29.21 0)
+			(hide yes)
+			(show_name no)
+			(do_not_autoplace no)
+			(effects
+				(font
+					(size 1.27 1.27)
+				)
+			)
+		)
 		(pin "2"
 		)
@@
 			)
 		)
+		(property "LCSC Part" "A"
+			(at 80.01 81.28 90)
+			(hide yes)
+			(show_name no)
+			(do_not_autoplace no)
+			(effects
+				(font
+					(size 1.27 1.27)
+				)
+			)
+		)
 		(pin "2"
 		)
@@
 			)
 		)
+		(property "LCSC Part" "A"
+			(at 106.68 110.49 0)
+			(hide yes)
+			(show_name no)
+			(do_not_autoplace no)
+			(effects
+				(font
+					(size 1.27 1.27)
+				)
+			)
+		)
 		(pin "2"
 		)
@@
 			)
 		)
+		(property "LCSC Part" "A"
+			(at 148.59 83.82 90)
+			(hide yes)
+			(show_name no)
+			(do_not_autoplace no)
+			(effects
+				(font
+					(size 1.27 1.27)
+				)
+			)
+		)
 		(pin "2"
 		)
@@
 			)
 		)
+		(property "LCSC Part" "A"
+			(at 148.59 71.12 90)
+			(hide yes)
+			(show_name no)
+			(do_not_autoplace no)
+			(effects
+				(font
+					(size 1.27 1.27)
+				)
+			)
+		)
 		(pin "2"
 		)
@@
 			(hide yes)
 			(show_name no)
+			(do_not_autoplace no)
+			(effects
+				(font
+					(size 1.27 1.27)
+				)
+			)
+		)
+		(property "LCSC Part" "A"
+			(at 80.01 55.88 90)
+			(hide yes)
+			(show_name no)

Commit message: Update letter.kicad_sch
Parts:
- C1, C10, C2, C3, C4, C5, C6, C7, C8, C9: LCSC Part A -> C1000
Changed lines of the file:
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@@
 			)
 		)
-		(property "LCSC Part" "A"
+		(property "LCSC Part" "C1000"
 			(at 80.01 68.58 90)
 			(hide yes)
@@
 			)
 		)
-		(property "LCSC Part" "A"
+		(property "LCSC Part" "C1000"
 			(at 109.22 29.21 0)
 			(hide yes)
@@
 			)
 		)
-		(property "LCSC Part" "A"
+		(property "LCSC Part" "C1000"
 			(at 148.59 58.42 90)
 			(hide yes)
@@
 			)
 		)
-		(property "LCSC Part" "A"
+		(property "LCSC Part" "C1000"
 			(at 119.38 110.49 0)
 			(hide yes)
@@
 			)
 		)
-		(property "LCSC Part" "A"
+		(property "LCSC Part" "C1000"
 			(at 121.92 29.21 0)
 			(hide yes)
@@
 			)
 		)
-		(property "LCSC Part" "A"
+		(property "LCSC Part" "C1000"
 			(at 80.01 81.28 90)
 			(hide yes)
@@
 			)
 		)
-		(property "LCSC Part" "A"
+		(property "LCSC Part" "C1000"
 			(at 106.68 110.49 0)
 			(hide yes)
@@
 			)
 		)
-		(property "LCSC Part" "A"
+		(property "LCSC Part" "C1000"
 			(at 148.59 83.82 90)
 			(hide yes)
@@
 			)
 		)
-		(property "LCSC Part" "A"
+		(property "LCSC Part" "C1000"
 			(at 148.59 71.12 90)
 			(hide yes)
@@
 			)
 		)
-		(property "LCSC Part" "A"
+		(property "LCSC Part" "C1000"
 			(at 80.01 55.88 90)
 			(hide yes)
